File: PCB/Icey.kicad_pcb (KiCad board)
At the start: 4 copper layers, 68.7 x 53 mm, 114 parts, among them J1 Conn_01x12, J2 Conn_01x08, SW2 TS-1088-AR02016, SW3 TS-1088-AR02016, U1 AMS1117-1.2, U2 ICE40UP5K-SG48I, U3 MAX3421EETJ+T, U4 W25Q128JVSIQTR, U5 AMS1117-3.3, U6 FT2232HL, U8 FM-B2020RGBA-HG_C42421005, X1 X322512MSB4SI, X2 X322512MSB4SI

Commit message: checkpoint: pwr plane done
Parts:
- removed D1: SS14, easyeda2kicad:SMA_L4.2-W2.6-LS5.0-RD_1
- removed R41, R42, R43: 0, Capacitor_SMD:C_0603_1608Metric
- removed U8: FM-B2020RGBA-HG_C42421005, easyeda2kicad:LED-SMD_FM-B2020RGBA-HG
- added LED4: S4-3528RGBTA-A, easyeda2kicad:LED-SMD_4P-L3.2-W2.8-LS3.5-TL-1, F.Cu at (150.6, 83.6)
- moved TP3 60.7 mm to (166.7, 131.2)
- moved TP4 60.7 mm to (170.6, 131.2)
- moved TP5 60.7 mm to (178.5, 131.2)
- moved TP6 60.7 mm to (174.5, 131.2)
- moved JP7 50.0 mm to (174.1, 124.4)
- moved JP8 49.5 mm to (174.1, 127.0), turned to 180 degrees
- moved R35 41.1 mm to (138.3, 94.4), turned to 0 degrees
- moved USB2 37.6 mm to (184.2, 93.3), turned to 90 degrees
- moved U4 36.6 mm to (144.5, 96.4), turned to -90 degrees
- moved USB1 32.7 mm to (184.2, 103.8), turned to 90 degrees
- moved C1 32.0 mm to (175.4, 90.4), turned to 180 degrees
- moved R4 31.3 mm to (179.7, 91.7), turned to 180 degrees
- moved R3 30.9 mm to (179.3, 94.6), turned to 180 degrees
- moved U5 29.9 mm to (175.1, 85.6), turned to 180 degrees
- moved C27 29.5 mm to (148.8, 93.3), turned to 0 degrees
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Connections:
- J1 pad 11: VBUS -> +3V3
- J1 pad 12: +3V3 -> VBUS
- U2 pad 44: /USB_SCLK -> /SD_SCK
- U2 pad 45: /USB_MISO -> /SD_MISO
- U2 pad 48: /USB_MOSI -> /SD_MOSI
- U3 pad 13: /USB_SCLK -> /SD_SCK
- U3 pad 15: /USB_MISO -> /SD_MISO
- U3 pad 16: /USB_MOSI -> /SD_MOSI
- USB2 pad B4A9: Net-(D1-A) -> VBUS
Routing:
- net VBUS: track 0.00 -> 133.0 mm, vias 0 -> 8
- net +1V2: track 0.00 -> 86.7 mm, vias 0 -> 8
- net +3V3: track 0.00 -> 42.6 mm, vias 0 -> 31
- net /PER_D-: track 24.2 -> 5.96 mm
- net /PER_D+: track 24.3 -> 6.06 mm
- net /SD_MOSI: track 17.6 -> 0.00 mm
- net /SD_SCK: track 11.5 -> 0.00 mm, vias 2 -> 0
- net Net-(U6-VPHY): track 10.6 -> 0.00 mm
- net /PROG_D+: track 51.0 -> 61.3 mm, vias 2 -> 0
- net Net-(U6-VPLL): track 10.1 -> 0.00 mm
- net /GREEN: track 0.00 -> 9.82 mm
- net Net-(F1-Pad1): track 0.00 -> 8.78 mm
- net /RED: track 0.00 -> 8.72 mm
- net /BLUE: track 0.00 -> 8.60 mm
- net Net-(U3-D+): track 2.10 -> 9.38 mm
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- added copper zone on In2.Cu, net +1V2

Commit message: checkpoint: gnd plane done
Parts:
- moved TP6 53.4 mm to (121.5, 124.4)
- moved TP4 48.6 mm to (169.0, 82.6)
- moved TP3 8.60 mm to (175.3, 131.1)
- moved C4 0.50 mm to (171.6, 98.7)
Routing:
- net +1V2: track 86.7 -> 44.2 mm
- net VBUS: track 133.0 -> 157.5 mm
- net GND: track 0.00 -> 14.3 mm, vias 2 -> 71
- net +3V3: track 42.6 -> 43.6 mm, vias 31 -> 32
- net Net-(U3-VBCOMP): track 1.46 -> 1.96 mm

Commit message: mostly
Parts:
- moved LED4 34.2 mm to (135.1, 114.0)
- moved R35 8.54 mm to (143.2, 101.4), turned to 90 degrees
- moved C26 8.31 mm to (140.5, 90.9), turned to 90 degrees
- moved C27 7.10 mm to (142.1, 90.9), turned to 90 degrees
- moved U4 1.45 mm to (145.2, 95.1), turned to 0 degrees
- moved C37 0.45 mm to (126.9, 108.8)
- moved C38 0.45 mm to (130.2, 108.5)
- moved R36 0.05 mm to (158.3, 85.4), turned to 180 degrees
Routing:
- net /PROG_RX: track 0.00 -> 47.2 mm
- net /PROG_TX: track 0.00 -> 46.2 mm
- net /SD_CS: track 0.00 -> 43.9 mm, vias 0 -> 2
- net /SD_MOSI: track 0.00 -> 43.3 mm, vias 0 -> 2
- net /SCK: track 0.00 -> 41.0 mm, vias 0 -> 3
- net /SD_SCK: track 0.00 -> 40.6 mm, vias 0 -> 2
- net /SD_MISO: track 0.00 -> 40.4 mm, vias 0 -> 2
- net /MOSI: track 0.00 -> 39.5 mm, vias 0 -> 2
- net /CS: track 0.00 -> 39.4 mm, vias 0 -> 1
- net /LED: track 0.00 -> 35.7 mm, vias 0 -> 2
- net /HSYNC: track 0.00 -> 34.6 mm, vias 0 -> 1
- net /VSYNC: track 0.00 -> 34.0 mm, vias 0 -> 1
- net /USB_INT: track 0.00 -> 33.3 mm, vias 0 -> 4
- net /USB_CS: track 0.00 -> 29.9 mm, vias 0 -> 2
- net /USB_RST: track 0.00 -> 29.3 mm, vias 0 -> 2
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
Commit message: pcb ready, needs art
Parts:
- added R41: 10K, Resistor_SMD:R_0603_1608Metric, F.Cu at (148.9, 98.6)
- added R42: 10K, Resistor_SMD:R_0603_1608Metric, F.Cu at (143.8, 88.0)
- added TP7: TestPoint, TestPoint:TestPoint_Pad_D2.0mm, F.Cu at (178.4, 128.0)
- R14, R15, R16, R17, R18, R19, R20, R21, R24, R25, R26, R27, R28, R29, R3, R30, R31, R32, R33, R34, R35, R36, R38, R39, R4, R40, R44, R45, R46, R47, R48, R5, R6, R9: footprint Capacitor_SMD:C_0603_1608Metric -> Resistor_SMD:R_0603_1608Metric
- moved JP5 56.1 mm to (169.7, 129.2), turned to -90 degrees
- moved JP3 55.4 mm to (164.6, 129.2), turned to -90 degrees
- moved JP4 54.3 mm to (167.2, 129.2), turned to -90 degrees
- moved R19 54.0 mm to (167.0, 131.7)
- moved JP2 53.6 mm to (162.1, 129.2), turned to -90 degrees
- moved JP1 52.8 mm to (159.6, 126.8), turned to -90 degrees
- moved JP6 51.1 mm to (169.6, 126.2)
- moved R36 24.8 mm to (133.6, 87.8), turned to 0 degrees
- moved R15 20.2 mm to (152.7, 100.3), turned to -90 degrees
- moved LED2 18.2 mm to (136.9, 87.8), turned to 180 degrees
- moved R14 17.1 mm to (154.2, 100.3), turned to -90 degrees
- moved R48 14.8 mm to (184.4, 122.7)
- moved R47 11.7 mm to (181.4, 122.7)
- moved R39 9.69 mm to (174.2, 115.2)
- moved R38 9.45 mm to (174.3, 113.7)
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Routing:
- net /creset_b: track 25.5 -> 108.8 mm, vias 2 -> 3
- net /MOSI: track 39.5 -> 117.6 mm, vias 2 -> 4
- net /MISO: track 29.2 -> 101.2 mm, vias 1 -> 3
- net /CDONE: track 20.5 -> 90.9 mm, vias 2 -> 4
- net /CS: track 39.4 -> 95.4 mm, vias 1 -> 3
- net /VCORE: track 0.00 -> 51.6 mm
- net /SCK: track 41.0 -> 77.6 mm, vias 3 -> 5
- net /SD_SCK: track 40.6 -> 73.0 mm, vias 2 -> 5
- net /SD_MISO: track 40.4 -> 71.9 mm, vias 2 -> 5
- net Net-(U2-IOB_25b_G3): track 0.00 -> 28.6 mm, vias 0 -> 2
- net /PROG_D-: track 61.2 -> 33.8 mm
- net Net-(U2-IOB_23b): track 0.00 -> 26.4 mm, vias 0 -> 2
- net /PROG_D+: track 61.3 -> 36.4 mm
- net Net-(U6-DM): track 1.87 -> 26.2 mm
- net Net-(U2-IOB_31b): track 0.00 -> 23.6 mm, vias 0 -> 2
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- added copper zone on B.Cu, net GND
- added copper zone on F.Cu, net GND

Commit message: done!!
Parts:
- moved JP1 2.45 mm to (159.5, 129.2)
Routing:
- net GND: track 17.7 -> 15.1 mm, vias 97 -> 98
- net /JTAG_TCK: track 4.80 -> 7.27 mm
- net /BUTTON: track 27.3 -> 25.0 mm
- net /PROG_TX: track 49.1 -> 50.8 mm
- net /ADBUS5: track 8.54 -> 6.88 mm
- net /LED: track 34.5 -> 32.9 mm
- net +3V3: track 44.3 -> 42.9 mm
- net /JTAG_TRST: track 9.63 -> 8.22 mm
- net /SD_MISO: track 71.9 -> 70.6 mm
- net /creset_b: track 108.8 -> 108.0 mm
- net /JTAG_TMS: track 8.91 -> 8.05 mm
- net Net-(U6-BDBUS3): track 3.63 -> 2.78 mm
- net /PROG_RX: track 51.0 -> 51.9 mm
- net Net-(U6-~{RESET}): track 3.10 -> 2.29 mm
- net /FLASH_HOLD: track 36.0 -> 35.2 mm
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Other:
- board text added: "1V2"
- board text added: "1V2 LDO"
- board text added: "3V3"
- board text added: "3V3 LDO"
- board text added: "CDONE"
- board text added: "CS"
- board text added: "FPGA"
- board text added: "GND"
- board text added: "HOLD"
- board text added: "IOB_13b"
- board text added: "IOB_16a"
- board text added: "IOT_42b"
- board text added: "IOT_43a"
- board text added: "IOT_44b"
- board text added: "IOT_45a"
- board text added: "IOT_46b"
- board text added: "IOT_48b"
- board text added: "IOT_49a"
- board text added: "IOT_50b"
- board text added: "IOT_51a"
- board text added: "Icey!!"
- board text added: "MICRO SD"
- board text added: "MISO"
- board text added: "MOSI"
- board text added: "PERIPHERAL"
- board text added: "PROG RX"
- board text added: "PROG TX"
- board text added: "PROGRAMMER"
- board text added: "QSPI FLASH"
- board text added: "RESET"
- board text added: "RGB LED"
- board text added: "SCK"
- board text added: "TCK"
- board text added: "TDI"
- board text added: "TDO"
- board text added: "TMS"
- board text added: "TRST"
- board text added: "USB HOST"
- board text added: "VBUS"
- board text added: "VCORE"
- board text added: "WP"
- board text added: "by darsh!!"
- board text added: "find the source at github.com/darshg321/Icey!"
- board text added: "v1.0"
